File: hw/YellowMotorEncoder.sch (EAGLE design)
At the start: 20 parts, among them P1 M1

Commit message: Make many improvements according testing v1.0 and v1.1 boards
- increase version number from v1.1 to v1.2
- decrease width of board from 22.4 to 22.2 mm
- move all parts to corresponding position with respect to the board center
- move hall sensor:
  - Y axis: 0.25 mm closer to the center of board (distance between both sensors is -0.5 mm)
  - X axis: 0.8 mm in motor direction
- improve documetation texts
  - increase size, add some labels
Other:
- note added: "v1.2"
- note removed: "v1.1"
Changed lines of the file:
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@@
 CC BY-SA 4.0</text>
 <text x="140.97" y="20.32" size="2.54" layer="97" font="vector" ratio="14">RobotikaBrno</text>
-<text x="171.45" y="5.08" size="2.54" layer="97" font="vector" ratio="14">v1.1</text>
+<text x="171.45" y="5.08" size="2.54" layer="97" font="vector" ratio="14">v1.2</text>
 <rectangle x1="135.370040625" y1="18.3900375" x2="135.583396875" y2="18.4002" layer="102"/>
 <rectangle x1="135.2278" y1="18.4002" x2="135.7256375" y2="18.41035625" layer="102"/>

Commit message: FourProbes
Parts:
- removed C2: 10n/50V, rcl:C-EUC0402
- removed JP1: (no value), pinhead:PINHD-1X6
- removed U$3: YELLOW_MOTOR, motor:YELLOW_MOTOR
- added C10: 20n/50V, rcl:C-EUC0402
- added C8, C9: 18p/50V, rcl:C-EUC0402
- added M1: MOTOR, motor:MOTOR
- added R6, R7: 47k, rcl:R-EU_R0402
- added U$4, U$5: MH253ESO, hall_sensor:MH253ESO
- added U1: SN74LVC2G86DCTR, SN74LVC2G86DCTR:SN74LVC2G86DCTR
- C1: value 10n/50V -> 20n/50V
- R1, R2, R3, R4, R5: device rcl:R-EU_R0603 -> rcl:R-EU_R0402
Connections:
- new net A0: C8.1, R6.1, U$4.OUT, U1.0B
- new net A1: C9.1, R7.1, U$5.OUT, U1.0A
- new net B0: C6.1, R4.1, U$1.OUT, U1.1B
- new net B1: C7.1, R5.1, U$2.OUT, U1.1A
- net A: now also U1.0Y; no longer C6.1, JP1.4, R4.1, U$1.OUT
- net B: now also U1.1Y; no longer C7.1, JP1.3, R5.1, U$2.OUT
- net GND: now also C10.2, C8.2, C9.2, U$4.GND, U$5.GND, U1.VCC; no longer C2.2, JP1.2
- net M+: now also M1.P$1; no longer JP1.6, U$3.P$2
- net M-: now also M1.P$2; no longer JP1.1, U$3.P$1
- net VCC: now also C10.1, R6.2, R7.2, U$4.VCC, U$5.VCC, U1.GND; no longer C2.1, JP1.5
Other:
- note added: "v1.3"
- note removed: "v1.2"
- moved on the sheet: C1, C3, C4, C5, C6, C7, LED_A, LED_B, LED_POWER, P1, R1, R2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

Commit message: ochrany
Parts:
- added C2: 20n/50V, rcl_upravena:C-EUC0402
- added Q1: FDN360P, transistor-power:FDN360P
- added R8, R9: 200, rcl_upravena:R-EU_R0402
- C1, C10, C6, C7, C8, C9: device rcl:C-EUC0402 -> rcl_upravena:C-EUC0402
- M1: value MOTOR -> YELLOW_MOTORV2; device motor:MOTOR -> motor:YELLOW_MOTORV2
- R1, R2, R3, R4, R5, R6, R7: device rcl:R-EU_R0402 -> rcl_upravena:R-EU_R0402
Connections:
- new net !A: R2.1, R8.1, U1.1Y
- new net !B: R3.1, R9.1, U1.0Y
- new net N$1: P1.2, Q1.D
- net A: now also R8.2; no longer R2.1, U1.0Y
- net A0: now also U1.1B; no longer U1.0B
- net A1: now also U1.1A; no longer U1.0A
- net B: now also R9.2; no longer R3.1, U1.1Y
- net B0: now also U1.0B; no longer U1.1B
- net B1: now also U1.0A; no longer U1.1A
- net GND: now also C2.2, Q1.G, U1.GND; no longer U1.VCC
- net VCC: now also C2.1, Q1.S, U1.VCC; no longer P1.2, U1.GND
Other:
- moved on the sheet: U1
